File: ESPinsupressor/ESPChipPCB.kicad_pcb (KiCad board)
At the start: 2 copper layers, 45.3 x 75 mm, 23 parts, among them J1 Conn_01x02, J2 Conn_01x02, J4 Conn_01x02, J5 Conn_01x04, Q1 BPW40, Q2 BPW40, SW1 SW_Push, U1 ESP32-C3-WROOM-02

Commit message: fixes
Parts:
- moved J4 1.71 mm to (162.7, 96.2)
- moved J1 0.70 mm to (151.1, 110.6)
Routing:
- net /D+: track 18.9 -> 15.6 mm
- net GND: track 90.4 -> 92.2 mm
- net +3.3V: track 119.3 -> 121.1 mm
- net /D-: track 11.6 -> 9.96 mm
- net /SecondSensor: track 102.3 -> 101.6 mm
